File: exhaust-fan-portable_hardware/Electronics/exhaust-fan-portable/Sensors.kicad_sch (KiCad schematic)
At the start: 0 parts

Commit message: layed out rough schematic and added sensor comparison
Parts:
- added C10, C11: 100nF, symbol Device:C
- added U2: BME280, Package_LGA:Bosch_LGA-8_2.5x2.5mm_P0.65mm_ClockwisePinNumbering, symbol Sensor:BME280
Connections:
- new net +3V3: C10.2, C11.2, U2.6 (VDDIO), U2.8 (VDD)
- new net GND: C10.1, C11.1, U2.1 (GND), U2.7 (GND)
- new net SPI_CS: U2.2 (CSB)
- new net SPI_MISO: U2.5 (SDO)
- new net SPI_MOSI: U2.3 (SDI)
- new net SPI_SCK: U2.4 (SCK)

Commit message: fixed case design
Parts:
- C10, C11: footprint (none) -> Capacitor_SMD:C_0603_1608Metric_Pad1.08x0.95mm_HandSolder
Changed lines of the file:
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@@
 			)
 		)
-		(property "Footprint" ""
+		(property "Footprint" "Capacitor_SMD:C_0603_1608Metric_Pad1.08x0.95mm_HandSolder"
 			(at 139.7 53.0352 0)
 			(effects
@@
 			)
 		)
-		(property "Footprint" ""
+		(property "Footprint" "Capacitor_SMD:C_0603_1608Metric_Pad1.08x0.95mm_HandSolder"
 			(at 139.7 63.1952 0)
 			(effects
